File: src/pcb/osuPad/osuPad.kicad_pcb (KiCad board)
At the start: 2 copper layers, 66 x 81 mm, 11 parts, among them SW1 SW_Push, SW2 SW_Push, SW3 SW_Push, SW4 SW_Push, SW5 SW_Push, SW6 SW_Push, SW7 SW_Push, SW8 SW_Push, SW9 SW_Push, U1 XIAO-RP2040-DIP

Commit message: update model and image
Routing:
- net GND: track 247.5 -> 249.1 mm
- net Net-(U1-GPIO28/ADC2/A2): track 67.4 -> 66.3 mm
- net Net-(U1-GPIO27/ADC1/A1): track 84.6 -> 83.6 mm
- net Net-(U1-GPIO26/ADC0/A0): track 103.9 -> 103.0 mm
- net Net-(U1-GPIO1/RX): track 67.3 -> 66.4 mm
- net Net-(U1-GPIO0/TX): track 16.9 -> 16.1 mm
- net Net-(U1-GPIO2/SCK): track 47.9 -> 47.2 mm
- net Net-(U1-GPIO29/ADC3/A3): track 76.9 -> 76.2 mm

Commit message: update firmware
Routing:
- net GND: track 249.1 -> 246.1 mm, vias 1 -> 2
- net Net-(U1-GPIO28/ADC2/A2): track 66.3 -> 66.2 mm, vias 2 -> 0
- net Net-(U1-GPIO27/ADC1/A1): track 83.6 -> 83.5 mm, vias 2 -> 0
- net Net-(U1-GPIO26/ADC0/A0): vias 2 -> 0
