File: PCB/osuPad/osuPad.kicad_sch (KiCad schematic)
At the start: 11 parts, among them SW1 SW_Push, SW2 SW_Push, SW3 SW_Push, SW4 SW_Push, SW5 SW_Push, SW6 SW_Push, SW7 SW_Push, SW8 SW_Push, SW9 SW_Push, U1 XIAO-RP2040-DIP

Commit message: add journal
Other:
- title: (none) -> osuPad Schematic
Changed lines of the file:
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@@
 	(generator_version "9.0")
 	(paper "A4")
+	(title_block
+		(title "osuPad Schematic")
+		(date "2025-06-14")
+		(rev "1")
+	)
 	(junction
 		(at 74.93 123.19)
